Commit message: added cone inertia

File: src/my_robot_description/urdf/common_properties.xacro (robot description, xacro)
@@ -28,3 +28,12 @@
     </inertial>
 </xacro:macro>
+<xacro:macro name="cone_inertia" params="m r o_xyz o_rpy">
+    <inertial>
+        <mass value="${m}" />
+        <origin xyz="${o_xyz}" rpy="${o_rpy}" />
+        <inertia ixx="${(3/10 * m * r * r)}" ixy="0" ixz="0"
+                iyy="${3/10 * m * r * r}" iyz="0"
+                izz="${3/10 * m * r * r}" />
+    </inertial>
+</xacro:macro>
 </robot>

Commit message: Removed fool bot folders as testing for these should be done in a new branch, colcon build does not work until CMake.txt is added properly for these files

File: src/my_robot_description/urdf/common_properties.xacro (robot description, xacro)
@@ -1,39 +1,3 @@
-<?xml version="1.0"?>
-<robot xmlns:xacro="http://www.ros.org/wiki/xacro">
-<xacro:macro name="box_inertia" params="m x y z o_xyz o_rpy">
-    <inertial>
-        <mass value="${m}" />
-        <origin xyz="${o_xyz}" rpy="${o_rpy}" />
-        <inertia ixx="${(m/12) * (y*y + z*z)}" ixy="0" ixz="0"
-                 iyy="${(m/12) * (x*x + z*z)}" iyz="0"
-                 izz="${(m/12) * (x*x + y*y)}" />
-    </inertial>
-</xacro:macro>
-<xacro:macro name="cylinder_inertia" params="m r l o_xyz o_rpy">
-    <inertial>
-        <mass value="${m}" />
-        <origin xyz="${o_xyz}" rpy="${o_rpy}" />
-        <inertia ixx="${(m/12) * (3*r*r + l*l)}" ixy="0" ixz="0"
-                 iyy="${(m/12) * (3*r*r + l*l)}" iyz="0"
-                 izz="${(m/2) * (r*r)}" />
-    </inertial>
-</xacro:macro>
-<xacro:macro name="sphere_inertia" params="m r o_xyz o_rpy">
-    <inertial>
-        <mass value="${m}" />
-        <origin xyz="${o_xyz}" rpy="${o_rpy}" />
-        <inertia ixx="${(2/5) * m * r * r}" ixy="0" ixz="0"
-                 iyy="${(2/5) * m * r * r}" iyz="0"
-                 izz="${(2/5) * m * r * r}" />
-    </inertial>
-</xacro:macro>
-<xacro:macro name="cone_inertia" params="m r o_xyz o_rpy">
-    <inertial>
-        <mass value="${m}" />
-        <origin xyz="${o_xyz}" rpy="${o_rpy}" />
-        <inertia ixx="${(3/10 * m * r * r)}" ixy="0" ixz="0"
-                iyy="${3/10 * m * r * r}" iyz="0"
-                izz="${3/10 * m * r * r}" />
-    </inertial>
-</xacro:macro>
-</robot>
+version https://git-lfs.github.com/spec/v1
+oid sha256:54092c25794c49ae4d714612b257332f7244b2b5b3910524c5bbf357d0faeb7d
+size 1483

File: src/my_robot_description/urdf/mobile_base_gazebo.xacro (robot description, xacro)
@@ -1,23 +1,3 @@
-<?xml version="1.0"?>
-<robot xmlns:xacro="http://www.ros.org/wiki/xacro">
-    <gazebo reference="caster_wheel_link">
-        <mu1 value="0.1" />
-        <mu2 value="0.1" />
-    </gazebo>
-    <gazebo>
-        <plugin filename="gz-sim-diff-drive-system" name="gz::sim::systems::DiffDrive">
-            <left_joint>base_left_wheel_joint</left_joint>
-            <right_joint>base_right_wheel_joint</right_joint>
-            <wheel_separation>0.45</wheel_separation>
-            <wheel_radius>0.1</wheel_radius>
-            <frame_id>odom</frame_id>
-            <child_frame_id>base_footprint</child_frame_id>
-        </plugin>
-    </gazebo>
-    <gazebo>
-        <plugin filename="gz-sim-joint-state-publisher-system" name="gz::sim::systems::JointStatePublisher">
-            <joint_name>base_left_wheel_joint</joint_name>
-            <joint_name>base_right_wheel_joint</joint_name>
-        </plugin>
-    </gazebo>
-</robot>
+version https://git-lfs.github.com/spec/v1
+oid sha256:86f925b2d48263eb6769d4687412db50af3a3a51f0d9aebbf95fa867db638064
+size 923

File: src/my_robot_description/urdf/my_robot.urdf.xacro (robot description, xacro)
@@ -1,103 +1,3 @@
-<?xml version="1.0"?>
-<robot name="my_robot" xmlns:xacro="http://www.ros.org/wiki/xacro">
-    <xacro:include filename="common_properties.xacro" />
-    <xacro:include filename="mobile_base_gazebo.xacro" />
-    <xacro:property name="base_length" value="0.6" />
-    <xacro:property name="base_width" value="0.4" />
-    <xacro:property name="base_height" value="0.2" />
-    <xacro:property name="wheel_radius" value="0.1" />
-    <xacro:property name="wheel_length" value="0.05" />
-    <material name="blue">
-        <color rgba="0 0 0.5 1" />
-    </material>
-    <material name="grey">
-        <color rgba="0.5 0.5 0.5 1" />
-    </material>
-    <link name="base_footprint" />
-    <link name="base_link">
-        <visual>
-            <geometry>
-                <box size="${base_length} ${base_width} ${base_height}" />
-            </geometry>
-            <origin xyz="0 0 ${base_height / 2.0}" rpy="0 0 0" />
-            <material name="blue" />
-        </visual>
-        <collision>
-            <geometry>
-                <box size="${base_length} ${base_width} ${base_height}" />
-            </geometry>
-            <origin xyz="0 0 ${base_height / 2.0}" rpy="0 0 0" />
-        </collision>
-        <xacro:box_inertia m="5.0" x="${base_length}" y="${base_width}" z="${base_height}" o_xyz="0 0 ${base_height / 2.0}" o_rpy="0 0 0" />
-    </link>
-    <link name="right_wheel_link">
-        <visual>
-            <geometry>
-                <cylinder radius="${wheel_radius}" length="${wheel_length}" />
-            </geometry>
-            <origin xyz="0 0 0" rpy="${pi / 2.0} 0 0" />
-            <material name="grey" />
-        </visual>
-        <collision>
-            <geometry>
-                <sphere radius="${wheel_radius}" />
-            </geometry>
-            <origin xyz="0 0 0" rpy="0 0 0" />
-        </collision>
-        <xacro:cylinder_inertia m="1.0" r="${wheel_radius}" l="${wheel_length}" o_xyz="0 0 0" o_rpy="${pi / 2.0} 0 0" />
-    </link>
-    <link name="left_wheel_link">
-        <visual>
-            <geometry>
-                <cylinder radius="${wheel_radius}" length="${wheel_length}" />
-            </geometry>
-            <origin xyz="0 0 0" rpy="${pi / 2.0} 0 0" />
-            <material name="grey" />
-        </visual>
-        <collision>
-            <geometry>
-                <sphere radius="${wheel_radius}" />
-            </geometry>
-            <origin xyz="0 0 0" rpy="0 0 0" />
-        </collision>
-        <xacro:cylinder_inertia m="1.0" r="${wheel_radius}" l="${wheel_length}" o_xyz="0 0 0" o_rpy="${pi / 2.0} 0 0" />
-    </link>
-    <link name="caster_wheel_link">
-        <visual>
-            <geometry>
-                <sphere radius="${wheel_radius / 2.0}" />
-            </geometry>
-            <origin xyz="0 0 0" rpy="0 0 0" />
-            <material name="grey" />
-        </visual>
-        <collision>
-            <geometry>
-                <sphere radius="${wheel_radius / 2.0}" />
-            </geometry>
-            <origin xyz="0 0 0" rpy="0 0 0" />
-        </collision>
-        <xacro:sphere_inertia m="0.5" r="${wheel_radius / 2.0}" o_xyz="0 0 0" o_rpy="0 0 0" />
-    </link>
-    <joint name="base_joint" type="fixed">
-        <parent link="base_footprint" />
-        <child link="base_link" />
-        <origin xyz="0 0 ${wheel_radius}" rpy="0 0 0" />
-    </joint>
-    <joint name="base_right_wheel_joint" type="continuous">
-        <parent link="base_link" />
-        <child link="right_wheel_link" />
-        <origin xyz="${-base_length / 4.0} -0.225 0" rpy="0 0 0" />
-        <axis xyz="0 1 0" />
-    </joint>
-    <joint name="base_left_wheel_joint" type="continuous">
-        <parent link="base_link" />
-        <child link="left_wheel_link" />
-        <origin xyz="${-base_length /4.0} 0.225 0" rpy="0 0 0" />
-        <axis xyz="0 1 0" />
-    </joint>
-    <joint name="base_caster_wheel_joint" type="fixed">
-        <parent link="base_link" />
-        <child link="caster_wheel_link" />
-        <origin xyz="${base_length / 3.0} 0 -0.05" rpy="0 0 0" />
-    </joint>
-</robot>
+version https://git-lfs.github.com/spec/v1
+oid sha256:052c5ce14631bd07c441c8e955869eb1f4d686aa848b4ff74efac2bcbcaecd17
+size 4043

File: src/my_robot_description/urdf/pusharm.urdf.xacro (robot description, xacro)
@@ -1,51 +1,3 @@
-<xml version="1.0" ?>
-<robot name="push_arm" xmlns:xacro="http://www.ros.org/wiki/xacro">
-    <xacro:property name="pusher_arm_radius" value="0.05" />
-    <xacro:property name="pursher_arm_length" value="0.3" />
-    <xacro:property name="pusher_length" value="0.1" />
-    <xacro:property name="pusher_width" value="0.3" />
-    <xacro:property name="pusher_height" value="0.25" />
-    <material name="blue">
-        <color rgba="0 0 0.5 1" />
-    </material>
-    <material name="grey">
-        <color rgba="0.5 0.5 0.5 1" />
-    </material>
-    <link name="pusher_arm_link">
-        <visual>
-            <geometry>
-                <cylinder radius="${pusher_arm_radius}" length="${pusher_arm_length}" />
-            </geometry>
-            <origin xyz="0 0 0" rpy="${pi / 2.0} 0 0" />
-            <material name="grey" />
-        </visual>
-        <collision>
-            <geometry>
-                <cylinder radius="${pusher_arm_radius}" length="${pusher_arm_length}" />
-            </geometry>
-            <origin xyz="0 0 0" rpy="0 0 0" />
-        </collision>
-        <xacro:cylinder_inertia m="3.0" r="${pusher_arm_radius}" l="${pusher_arm_length}" o_xyz="0 0 0" o_rpy="${pi / 2} 0 0" />
-    </link>
-    <link name="pusher_link">
-        <visual>
-            <geometry>
-                <box size="${pusher_length} ${pusher_width} ${pusher_height}" />
-            </geometry>
-            <origin xyz="0 0 ${pusher_height/2}" rpy="0 0 0" />
-            <material name="grey" />
-        </visual>
-        <collision>
-            <geometry>
-                <box size="${pusher_length} ${pusher_width} ${pusher_height}" />
-            </geometry>
-            <origin xyz="0 0 ${pusher_height/2}" rpy="0 0 0" />
-        </collision>
-        <xacro:box_inertia m="2.0" x="${pusher_length}" y="${pusher_width}" z="${pusher_height}" o_xyz="0 0 ${pusher_height/2}" o_rpy="0 0 0" />
-    </link>
-    <joint name="pusher_pusher_arm_joint" type="fixed">
-        <parent link="pusher_arm_link" />
-        <child link="pusher_link" />
-        <origin xyz="0 0 ${-pusher_arm_length}" rpy="0 0 0" />
-    </joint>
-</robot>
+version https://git-lfs.github.com/spec/v1
+oid sha256:b47934370f5b6fe2f97ef3e607804407a1ad8188103d018f3d662c68f6ef41ec
+size 2116

File: src/my_robot_description/urdf/test.urdf.xacro (robot description, xacro)
@@ -1,217 +1,3 @@
-<?xml version="1.0"?>
-<robot name="test" xmlns:xacro="http://www.ros.org/wiki/xacro">
-<!--Please do not open this robot, this is for testing purposes only. Adding various tags and such to figure out what the different properties actually do-->
-<!--Xacro allows to add in variables, as seen below-->
-<!--INclude Xacro packages-->
-    <xacro:include filename="common_properties.xacro" />
-    <xacro:include filename="mobile_base_gazebo.xacro" />
-<!--Note - you can define more complex components in their own .xacro file to add to the robot file-->
-<!--Defining some xacro variables. Defined as xacro:property. Give a name and a value in order to use elsewhere. Changing here will adjust in the whole file.-->
-    <xacro:property name="base_length" value="0.6" />
-    <xacro:property name="base_width" value="0.4" />
-    <xacro:property name="base_height" value="0.2" />
-    <xacro:property name="wheel_radius" value="0.1" />
-    <xacro:property name="wheel_length" value="0.05" />
-    <xacro:property name="pusher_arm_radius" value="0.025" />
-    <xacro:property name="pusher_arm_length" value="0.4" />
-    <xacro:property name="pusher_length" value="0.1" />
-    <xacro:property name="pusher_width" value="0.3" />
-    <xacro:property name="pusher_height" value="0.1" />
-<!--Materials defied here, no need for exceptional appearance. Color is fine to save resources-->
-    <material name="blue">
-        <color rgba="0 0 0.5 1" />
-    </material>
-    <material name="grey">
-        <color rgba="0.5 0.5 0.5 1" />
-    </material>
-    <link name="base_footprint" /> <!--Self closing link tag, no properties-->
-    <!--Link tags here. Links are physical structures in the robot. Joints connect links, can be moveable or immovable-->
-    <!--Put all links first and then add joints to keep track-->
-    <link name="base_link">
-        <visual>
-            <geometry>
-                <box size="${base_length} ${base_width} ${base_height}" />
-            </geometry>
-            <origin xyz = "0 0 ${base_height / 2}" rpy="0 0 0" /> <!--Define origin of the shape - set to center of object-->
-            <material name="blue" /> <!--Xacro defined the material, line 15. Reusing the name calls back to the predefined variable, allowing you to save time and shorthand-->
-        </visual>
-        <collision>
-            <geometry>
-                <box size="${base_length} ${base_width} ${base_height}" />
-            </geometry>
-            <origin xyz = "0 0 ${base_height}/2" rpy="0 0 0" />
-        </collision>
-        <!--Generally, collision and visual will be the same. The exception is the wheel which uses a sphere collision rather than a cylinder, as it behaves oddly otherwise.-->
-        <xacro:box_inertia m="5.0" x="${base_length}" y="${base_width}" z="${base_height}" o_xyz="0 0 ${base_height / 2.0}" o_rpy="0 0 0" />
-        <!--Add inertia - taken from common_properties.xacro, predefined. You can define this on your own, but using predefined information is best for now until you understand-->
-    </link>
-    <!--My first item that I add-->
-    <link name="drill_cone_link">
-        <visual>
-            <geometry>
-                <mesh filename="package://my_robot_description/meshes/cone(blender).stl" scale="1 1 1"/>
-            </geometry>
-            <origin xyz = "0 0 0" rpy="0 ${pi/2} 0" />
-            <material name="grey" />
-        </visual>
-        <collision>
-            <geometry>
-                <mesh filename="package://my_robot_description/meshes/cone(blender).stl" scale = "1 1 1" />
-            </geometry>
-            <origin xyz = "0 0 0" rpy="0 ${pi/2} 0" />
-        </collision>
-        <xacro:cylinder_inertia m="1.0" r="${wheel_radius}" l="${base_length}" o_xyz="0 0 0" o_rpy="0 ${pi/2} 0" />
-    </link>
-    <link name="right_wheel_link">
-        <visual>
-            <geometry>
-                <cylinder radius="${wheel_radius}" length="${wheel_length}" /> <!--Length is the height of the cylinder-->
-            </geometry>
-            <origin xyz="0 0 0" rpy="${pi / 2.0} 0 0" /> <!--Rotation done in radians, thus in reference to PI-->
-            <material name="grey" />
-        </visual>
-        <collision>
-            <geometry>
-                <sphere radius="${wheel_radius}" />
-            </geometry>
-            <origin xyz="0 0 0" rpy="0 0 0" />
-        </collision>
-        <xacro:cylinder_inertia m="1.0" r="${wheel_radius}" l="${wheel_length}" o_xyz="0 0 0" o_rpy="${pi / 2.0} 0 0" />
-    </link>
-        <link name="left_wheel_link">
-        <visual>
-            <geometry>
-                <cylinder radius="${wheel_radius}" length="${wheel_length}" />
-            </geometry>
-            <origin xyz="0 0 0" rpy="${pi / 2.0} 0 0" />
-            <material name="grey" />
-        </visual>
-        <collision>
-            <geometry>
-                <sphere radius="${wheel_radius}" />
-            </geometry>
-            <origin xyz="0 0 0" rpy="0 0 0" />
-        </collision>
-        <xacro:cylinder_inertia m="1.0" r="${wheel_radius}" l="${wheel_length}" o_xyz="0 0 0" o_rpy="${pi / 2.0} 0 0" />
-    </link>
-    <link name="caster_wheel_link">
-        <visual>
-            <geometry>
-                <sphere radius="${wheel_radius / 2.0}" />
-            </geometry>
-            <origin xyz="0 0 0" rpy="0 0 0" />
-            <material name="grey" />
-        </visual>
-        <collision>
-            <geometry>
-                <sphere radius="${wheel_radius / 2.0}" />
-            </geometry>
-            <origin xyz="0 0 0" rpy="0 0 0" />
-        </collision>
-        <xacro:sphere_inertia m="0.5" r="${wheel_radius / 2.0}" o_xyz="0 0 0" o_rpy="0 0 0" />
-    </link>
-    <!--<xacro:include filename="$(find my_robot_description)/urdf/pusharm.urdf.xacro">
-    <link name="arm1_link" />-->
-        <link name="pusher_arm_link">
-        <visual>
-            <geometry>
-                <cylinder radius="${pusher_arm_radius}" length="${pusher_arm_length}" />
-            </geometry>
-            <origin xyz="0 0 0" rpy="0 0 0" />
-            <material name="grey" />
-        </visual>
-        <collision>
-            <geometry>
-                <cylinder radius="${pusher_arm_radius}" length="${pusher_arm_length}" />
-            </geometry>
-            <origin xyz="0 0 0" rpy="0 0 0" />
-        </collision>
-        <xacro:cylinder_inertia m="3.0" r="${pusher_arm_radius}" l="${pusher_arm_length}" o_xyz="0 0 0" o_rpy="0 0 0" />
-    </link>
-    <link name="left_pusher_link">
-        <visual>
-            <geometry>
-                <box size="${pusher_length} ${pusher_width} ${pusher_height}" />
-            </geometry>
-            <origin xyz="0 0 ${pusher_height/2}" rpy="0 0 0" />
-            <material name="grey" />
-        </visual>
-        <collision>
-            <geometry>
-                <box size="${pusher_length} ${pusher_width} ${pusher_height}" />
-            </geometry>
-            <origin xyz="0 0 ${pusher_height/2}" rpy="0 0 0" />
-        </collision>
-        <xacro:box_inertia m="2.0" x="${pusher_length}" y="${pusher_width}" z="${pusher_height}" o_xyz="0 0 ${pusher_height/2}" o_rpy="0 0 0" />
-    </link>
-    <link name="right_pusher_link">
-        <visual>
-            <geometry>
-                <box size="${pusher_length} ${pusher_width} ${pusher_height}" />
-            </geometry>
-            <origin xyz="0 0 ${pusher_height/2}" rpy="0 0 0" />
-            <material name="grey" />
-        </visual>
-        <collision>
-            <geometry>
-                <box size="${pusher_length} ${pusher_width} ${pusher_height}" />
-            </geometry>
-            <origin xyz="0 0 ${pusher_height/2}" rpy="0 0 0" />
-        </collision>
-        <xacro:box_inertia m="2.0" x="${pusher_length}" y="${pusher_width}" z="${pusher_height}" o_xyz="0 0 ${pusher_height/2}" o_rpy="0 0 0" />
-    </link>
-    <!--Joints here-->
-    <!--Joints attach links to each other. DIfferent joint types cause different behaviours. I.E "fixed" disallows movement, would be like welding. COntinuous allows rotation forever. So on.-->
-    <!--Origins are where the joint connects the different links - very important to give space for rotation-->
-    <joint name="base_joint" type="fixed">
-        <parent link="base_footprint" /> <!--Parent is what child is attached to - any rotation will be done as such-->
-        <child link="base_link" />
-        <origin xyz="0 0 ${wheel_radius}" rpy="0 0 0" />
-    </joint>
-    <!--My first joint, attaching drill to chassis-->
-    <joint name="base_drill_cone_joint" type="continuous">
-        <parent link="base_link" />
-        <child link="drill_cone_link" />
-        <origin xyz="${base_length} 0 ${wheel_radius}" rpy="0 0 0" />
-        <axis xyz="1 0 0" />
-    </joint>
-    <joint name="base_right_wheel_joint" type="continuous">
-        <parent link="base_link" />
-        <child link="right_wheel_link" />
-        <origin xyz="${-base_length / 4.0} -0.225 0" rpy="0 0 0" />
-        <axis xyz="0 1 0" />
-    </joint>
-    <joint name="base_left_wheel_joint" type="continuous">
-        <parent link="base_link" />
-        <child link="left_wheel_link" />
-        <origin xyz="${-base_length /4.0} 0.225 0" rpy="0 0 0" />
-        <axis xyz="0 1 0" />
-    </joint>
-    <joint name="base_caster_wheel_joint" type="fixed">
-        <parent link="base_link" />
-        <child link="caster_wheel_link" />
-        <origin xyz="${base_length / 3.0} 0 -0.05" rpy="0 0 0" />
-    </joint>
-    <!--<joint name="base_arm1_joint" type="fixed">
-        <parent link="base_link" />
-        <child link="arm1_link" />
-        <origin xyz="${base_length/2} ${base_width/2 + pusher_arm_radius} 0" rpy="0 0 0" />
-    </joint>-->
-    <joint name="left_pusher_pusher_arm_joint" type="fixed">
-        <parent link="pusher_arm_link" />
-        <child link="left_pusher_link" />
-        <origin xyz="0 0 ${-pusher_arm_length+pusher_height}" rpy="0 0 0" />
-    </joint>
-    <joint name="right_pusher_pusher_arm_joint" type="fixed">
-        <parent link="pusher_arm_link" />
-        <child link="right_pusher_link" />
-        <origin xyz="0 0 ${pusher_arm_length-pusher_height*2}" rpy="0 0 0" />
-    </joint>
-    <joint name="arm_base_link" type="prismatic">
-        <parent link="base_link" />
-        <child link="pusher_arm_link" />
-        <origin xyz="0 0 ${pusher_length/2 + base_height}" rpy="0 -1.571 1.571" />
-        <axis xyz="0 0 1" />
-        <limit lower="${-pusher_arm_length}" upper="${pusher_arm_length}" effort="20" velocity="0.5" />
-    </joint>
-</robot>
+version https://git-lfs.github.com/spec/v1
+oid sha256:abcbfda87ba8d4d23dcb4a532a6b1124c7c5abf773a9186fa584c9ecf082eb2d
+size 10488
