Commit message: Removed fool bot folders as testing for these should be done in a new branch, colcon build does not work until CMake.txt is added properly for these files

File: src/my_robot_description/urdf/untested.urdf.xacro (robot description, xacro)
@@ -1,76 +1,3 @@
-<?xml version="1.0"?>
-<robot name="my_robot" xmlns:xacro="http://www.ros.org/wiki/xacro">
-    <xacro:include filename="common_properties.xacro" />
-    <xacro:include filename="mobile_base_gazebo.xacro" />
-    <xacro:property name="base_length" value="0.6" />
-    <xacro:property name="base_width" value="0.4" />
-    <xacro:property name="base_height" value="0.2" />
-    <xacro:property name="wheel_radius" value="0.1" />
-    <xacro:property name="wheel_length" value="0.05" />
-    <xacro:property name="pusher_arm_radius" value="0.05" />
-    <xacro:property name="pursher_arm_length" value="0.3" />
-    <xacro:property name="pusher_length" value="0.1" />
-    <xacro:property name="pusher_width" value="0.3" />
-    <xacro:property name="pusher_height" value="0.25" />
-    <!--TODO: Make pusher independant file to add multiple on robot-->
-    <material name="blue">
-        <color rgba="0 0 0.5 1" />
-    </material>
-    <material name="grey">
-        <color rgba="0.5 0.5 0.5 1" />
-    </material>
-    <link name="base_footprint" />
-    <link name="base_link">
-        <visual>
-            <geometry>
-                <box size="${base_length} ${base_width} ${base_height}" />
-            </geometry>
-            <origin xyz="0 0 ${base_height / 2.0}" rpy="0 0 0" />
-            <material name="blue" />
-        </visual>
-        <collision>
-            <geometry>
-                <box size="${base_length} ${base_width} ${base_height}" />
-            </geometry>
-            <origin xyz="0 0 ${base_height / 2.0}" rpy="0 0 0" />
-        </collision>
-        <xacro:box_inertia m="5.0" x="${base_length}" y="${base_width}" z="${base_height}" o_xyz="0 0 ${base_height / 2.0}" o_rpy="0 0 0" />
-    </link>
-    <link name="pusher_arm_link">
-        <visual>
-            <geometry>
-                <cylinder radius="${pusher_arm_radius}" length="${pusher_arm_length}" />
-            </geometry>
-            <origin xyz="0 0 0" rpy="${pi / 2.0} 0 0" />
-            <material name="grey" />
-        </visual>
-        <collision>
-            <geometry>
-                <cylinder radius="${pusher_arm_radius}" length="${pusher_arm_length}" />
-            </geometry>
-            <origin xyz="0 0 0" rpy="0 0 0" />
-        </collision>
-        <xacro:cylinder_inertia m="3.0" r="${pusher_arm_radius}" l="${pusher_arm_length}" o_xyz="0 0 0" o_rpy="${pi / 2} 0 0" />
-    </link>
-    <link name="pusher_link">
-        <visual>
-            <geometry>
-                <box size="${pusher_length} ${pusher_width} ${pusher_height}" />
-            </geometry>
-            <origin xyz="0 0 ${pusher_height/2}" rpy="0 0 0" />
-            <material name="grey" />
-        </visual>
-        <collision>
-            <geometry>
-                <box size="${pusher_length} ${pusher_width} ${pusher_height}" />
-            </geometry>
-            <origin xyz="0 0 ${pusher_height/2}" rpy="0 0 0" />
-        </collision>
-        <xacro:box_inertia m="2.0" x="${pusher_length}" y="${pusher_width}" z="${pusher_height}" o_xyz="0 0 ${pusher_height/2}" o_rpy="0 0 0" />
-    </link>
-    <joint name="pusher_pusher_arm_joint" type="fixed">
-        <parent link="pusher_arm_link" />
-        <child link="pusher_link" />
-        <origin xyz="0 0 ${-pusher_arm_length}" rpy="0 0 0" />
-    </joint>
-</robot>
+version https://git-lfs.github.com/spec/v1
+oid sha256:ed87b03c991cf55d6c7aa33cd8e06299dd8a1a1d30e8fe97d1804832cc72e622
+size 3288
