Commit message: Fixed simple_test file so now it launches with launch command

File: install/my_robot_description/share/my_robot_description/urdf/my_robot.urdf.xacro (robot description, xacro)
@@ -1,6 +1,11 @@
 <?xml version="1.0"?>
-<robot name="my_robot" xmlns:xacro="http://www.ros.org/wiki/xacro">
+<robot name="test" xmlns:xacro="http://www.ros.org/wiki/xacro">
+<!--Took code from test to use here, do not use test.urdf.xacro-->
+<!--Xacro allows to add in variables, as seen below-->
+<!--INclude Xacro packages-->
     <xacro:include filename="common_properties.xacro" />
     <xacro:include filename="mobile_base_gazebo.xacro" />
+<!--Note - you can define more complex components in their own .xacro file to add to the robot file-->
+<!--Defining some xacro variables. Defined as xacro:property. Give a name and a value in order to use elsewhere. Changing here will adjust in the whole file.-->
     <xacro:property name="base_length" value="0.6" />
     <xacro:property name="base_width" value="0.4" />
@@ -8,4 +13,10 @@
     <xacro:property name="wheel_radius" value="0.1" />
     <xacro:property name="wheel_length" value="0.05" />
+    <xacro:property name="pusher_arm_radius" value="0.025" />
+    <xacro:property name="pusher_arm_length" value="0.4" />
+    <xacro:property name="pusher_length" value="0.1" />
+    <xacro:property name="pusher_width" value="0.3" />
+    <xacro:property name="pusher_height" value="0.1" />
+<!--Materials defied here, no need for exceptional appearance. Color is fine to save resources-->
     <material name="blue">
         <color rgba="0 0 0.5 1" />
@@ -14,13 +25,7 @@
         <color rgba="0.5 0.5 0.5 1" />
     </material>
-    <link name="base_footprint" />
-    <!--
-      _____ _    _           _____ _____ _____  _____
-     / ____| |  | |   /\    / ____/ ____|_   _|/ ____|
-    | |    | |__| |  /  \  | (___| (___   | | | (___
-    | |    |  __  | / /\ \  \___ \\___ \  | |  \___ \
-    | |____| |  | |/ ____ \ ____) |___) |_| |_ ____) |
-     \_____|_|  |_/_/    \_\_____/_____/|_____|_____/
-    -->
+    <link name="base_footprint" /> <!--Self closing link tag, no properties-->
+    <!--Link tags here. Links are physical structures in the robot. Joints connect links, can be moveable or immovable-->
+    <!--Put all links first and then add joints to keep track-->
     <link name="base_link">
         <visual>
@@ -28,6 +33,6 @@
                 <box size="${base_length} ${base_width} ${base_height}" />
             </geometry>
-            <origin xyz="0 0 ${base_height / 2.0}" rpy="0 0 0" />
-            <material name="blue" />
+            <origin xyz = "0 0 ${base_height / 2}" rpy="0 0 0" /> <!--Define origin of the shape - set to center of object-->
+            <material name="blue" /> <!--Xacro defined the material, line 15. Reusing the name calls back to the predefined variable, allowing you to save time and shorthand-->
         </visual>
         <collision>
@@ -35,19 +40,46 @@
                 <box size="${base_length} ${base_width} ${base_height}" />
             </geometry>
-            <origin xyz="0 0 ${base_height / 2.0}" rpy="0 0 0" />
-        </collision>
+            <origin xyz = "0 0 ${base_height}/2" rpy="0 0 0" />
+        </collision>
+        <!--Generally, collision and visual will be the same. The exception is the wheel which uses a sphere collision rather than a cylinder, as it behaves oddly otherwise.-->
         <xacro:box_inertia m="5.0" x="${base_length}" y="${base_width}" z="${base_height}" o_xyz="0 0 ${base_height / 2.0}" o_rpy="0 0 0" />
-    </link>
-    <!--
-     _____  _____ _____ _    _ _______  __          ___    _ ______ ______ _
-    |  __ \|_   _/ ____| |  | |__   __| \ \        / / |  | |  ____|  ____| |
-    | |__) | | || |  __| |__| |  | |     \ \  /\  / /| |__| | |__  | |__  | |
-    |  _  /  | || | |_ |  __  |  | |      \ \/  \/ / |  __  |  __| |  __| | |
-    | | \ \ _| || |__| | |  | |  | |       \  /\  /  | |  | | |____| |____| |____
-    |_|  \_\_____\_____|_|  |_|  |_|        \/  \/   |_|  |_|______|______|______|
-    -->
+        <!--Add inertia - taken from common_properties.xacro, predefined. You can define this on your own, but using predefined information is best for now until you understand-->
+    </link>
+    <!--My first item that I add-->
+    <link name="drill_cone_link">
+        <visual>
+            <geometry>
+                <mesh filename="package://my_robot_description/meshes/cone(blender).stl" scale="1 1 1"/>
+            </geometry>
+            <origin xyz = "0 0 0" rpy="0 ${pi/2} 0" />
+            <material name="grey" />
+        </visual>
+        <collision>
+            <geometry>
+                <mesh filename="package://my_robot_description/meshes/cone(blender).stl" scale = "1 1 1" />
+            </geometry>
+            <origin xyz = "0 0 0" rpy="0 ${pi/2} 0" />
+        </collision>
+        <xacro:cylinder_inertia m="1.0" r="${wheel_radius}" l="${base_length}" o_xyz="0 0 0" o_rpy="0 ${pi/2} 0" />
+    </link>
     <link name="right_wheel_link">
         <visual>
             <geometry>
+                <cylinder radius="${wheel_radius}" length="${wheel_length}" /> <!--Length is the height of the cylinder-->
+            </geometry>
+            <origin xyz="0 0 0" rpy="${pi / 2.0} 0 0" /> <!--Rotation done in radians, thus in reference to PI-->
+            <material name="grey" />
+        </visual>
+        <collision>
+            <geometry>
+                <sphere radius="${wheel_radius}" />
+            </geometry>
+            <origin xyz="0 0 0" rpy="0 0 0" />
+        </collision>
+        <xacro:cylinder_inertia m="1.0" r="${wheel_radius}" l="${wheel_length}" o_xyz="0 0 0" o_rpy="${pi / 2.0} 0 0" />
+    </link>
+        <link name="left_wheel_link">
+        <visual>
+            <geometry>
                 <cylinder radius="${wheel_radius}" length="${wheel_length}" />
             </geometry>
@@ -63,36 +95,4 @@
         <xacro:cylinder_inertia m="1.0" r="${wheel_radius}" l="${wheel_length}" o_xyz="0 0 0" o_rpy="${pi / 2.0} 0 0" />
     </link>
-    <!--
-     _      ______ ______ _______  __          ___    _ ______ ______ _
-    | |    |  ____|  ____|__   __| \ \        / / |  | |  ____|  ____| |
-    | |    | |__  | |__     | |     \ \  /\  / /| |__| | |__  | |__  | |
-    | |    |  __| |  __|    | |      \ \/  \/ / |  __  |  __| |  __| | |
-    | |____| |____| |       | |       \  /\  /  | |  | | |____| |____| |____
-    |______|______|_|       |_|        \/  \/   |_|  |_|______|______|______|
-    -->
-    <link name="left_wheel_link">
-        <visual>
-            <geometry>
-                <cylinder radius="${wheel_radius}" length="${wheel_length}" />
-            </geometry>
-            <origin xyz="0 0 0" rpy="${pi / 2.0} 0 0" />
-            <material name="grey" />
-        </visual>
-        <collision>
-            <geometry>
-                <sphere radius="${wheel_radius}" />
-            </geometry>
-            <origin xyz="0 0 0" rpy="0 0 0" />
-        </collision>
-        <xacro:cylinder_inertia m="1.0" r="${wheel_radius}" l="${wheel_length}" o_xyz="0 0 0" o_rpy="${pi / 2.0} 0 0" />
-    </link>
-    <!--
-      _____           _____ _______ ______ _____   __          ___    _ ______ ______ _
-     / ____|   /\    / ____|__   __|  ____|  __ \  \ \        / / |  | |  ____|  ____| |
-    | |       /  \  | (___    | |  | |__  | |__) |  \ \  /\  / /| |__| | |__  | |__  | |
-    | |      / /\ \  \___ \   | |  |  __| |  _  /    \ \/  \/ / |  __  |  __| |  __| | |
-    | |____ / ____ \ ____) |  | |  | |____| | \ \     \  /\  /  | |  | | |____| |____| |____
-     \_____/_/    \_\_____/   |_|  |______|_|  \_\     \/  \/   |_|  |_|______|______|______|
-    -->
     <link name="caster_wheel_link">
         <visual>
@@ -111,8 +111,68 @@
         <xacro:sphere_inertia m="0.5" r="${wheel_radius / 2.0}" o_xyz="0 0 0" o_rpy="0 0 0" />
     </link>
+    <!--<xacro:include filename="$(find my_robot_description)/urdf/pusharm.urdf.xacro">
+    <link name="arm1_link" />-->
+        <link name="pusher_arm_link">
+        <visual>
+            <geometry>
+                <cylinder radius="${pusher_arm_radius}" length="${pusher_arm_length}" />
+            </geometry>
+            <origin xyz="0 0 0" rpy="0 0 0" />
+            <material name="grey" />
+        </visual>
+        <collision>
+            <geometry>
+                <cylinder radius="${pusher_arm_radius}" length="${pusher_arm_length}" />
+            </geometry>
+            <origin xyz="0 0 0" rpy="0 0 0" />
+        </collision>
+        <xacro:cylinder_inertia m="3.0" r="${pusher_arm_radius}" l="${pusher_arm_length}" o_xyz="0 0 0" o_rpy="0 0 0" />
+    </link>
+    <link name="left_pusher_link">
+        <visual>
+            <geometry>
+                <box size="${pusher_length} ${pusher_width} ${pusher_height}" />
+            </geometry>
+            <origin xyz="0 0 ${pusher_height/2}" rpy="0 0 0" />
+            <material name="grey" />
+        </visual>
+        <collision>
+            <geometry>
+                <box size="${pusher_length} ${pusher_width} ${pusher_height}" />
+            </geometry>
+            <origin xyz="0 0 ${pusher_height/2}" rpy="0 0 0" />
+        </collision>
+        <xacro:box_inertia m="2.0" x="${pusher_length}" y="${pusher_width}" z="${pusher_height}" o_xyz="0 0 ${pusher_height/2}" o_rpy="0 0 0" />
+    </link>
+    <link name="right_pusher_link">
+        <visual>
+            <geometry>
+                <box size="${pusher_length} ${pusher_width} ${pusher_height}" />
+            </geometry>
+            <origin xyz="0 0 ${pusher_height/2}" rpy="0 0 0" />
+            <material name="grey" />
+        </visual>
+        <collision>
+            <geometry>
+                <box size="${pusher_length} ${pusher_width} ${pusher_height}" />
+            </geometry>
+            <origin xyz="0 0 ${pusher_height/2}" rpy="0 0 0" />
+        </collision>
+        <xacro:box_inertia m="2.0" x="${pusher_length}" y="${pusher_width}" z="${pusher_height}" o_xyz="0 0 ${pusher_height/2}" o_rpy="0 0 0" />
+    </link>
+    <!--Joints here-->
+    <!--Joints attach links to each other. DIfferent joint types cause different behaviours. I.E "fixed" disallows movement, would be like welding. COntinuous allows rotation forever. So on.-->
+    <!--Origins are where the joint connects the different links - very important to give space for rotation-->
     <joint name="base_joint" type="fixed">
-        <parent link="base_footprint" />
+        <parent link="base_footprint" /> <!--Parent is what child is attached to - any rotation will be done as such-->
         <child link="base_link" />
         <origin xyz="0 0 ${wheel_radius}" rpy="0 0 0" />
+    </joint>
+    <!--My first joint, attaching drill to chassis-->
+    <joint name="base_drill_cone_joint" type="continuous">
+        <parent link="base_link" />
+        <child link="drill_cone_link" />
+        <origin xyz="${base_length} 0 ${wheel_radius}" rpy="0 0 0" />
+        <axis xyz="1 0 0" />
     </joint>
     <joint name="base_right_wheel_joint" type="continuous">
@@ -133,3 +193,25 @@
         <origin xyz="${base_length / 3.0} 0 -0.05" rpy="0 0 0" />
     </joint>
+    <!--<joint name="base_arm1_joint" type="fixed">
+        <parent link="base_link" />
+        <child link="arm1_link" />
+        <origin xyz="${base_length/2} ${base_width/2 + pusher_arm_radius} 0" rpy="0 0 0" />
+    </joint>-->
+    <joint name="left_pusher_pusher_arm_joint" type="fixed">
+        <parent link="pusher_arm_link" />
+        <child link="left_pusher_link" />
+        <origin xyz="0 0 ${-pusher_arm_length+pusher_height}" rpy="0 0 0" />
+    </joint>
+    <joint name="right_pusher_pusher_arm_joint" type="fixed">
+        <parent link="pusher_arm_link" />
+        <child link="right_pusher_link" />
+        <origin xyz="0 0 ${pusher_arm_length-pusher_height*2}" rpy="0 0 0" />
+    </joint>
+    <joint name="arm_base_link" type="prismatic">
+        <parent link="base_link" />
+        <child link="pusher_arm_link" />
+        <origin xyz="0 0 ${pusher_length/2 + base_height}" rpy="0 -1.571 1.571" />
+        <axis xyz="0 0 1" />
+        <limit lower="${-pusher_arm_length}" upper="${pusher_arm_length}" effort="20" velocity="0.5" />
+    </joint>
 </robot>

Commit message: Began adding features to simple_test world, temporarily removed pusher arms from my_robot

File: install/my_robot_description/share/my_robot_description/urdf/my_robot.urdf.xacro (robot description, xacro)
@@ -47,5 +47,6 @@
     </link>
     <!--My first item that I add-->
-    <link name="drill_cone_link">
+    <!-- Drill does not need to be in the file until I can get the mesh import working -->
+    <!-- <link name="drill_cone_link">
         <visual>
             <geometry>
@@ -62,5 +63,5 @@
         </collision>
         <xacro:cylinder_inertia m="1.0" r="${wheel_radius}" l="${base_length}" o_xyz="0 0 0" o_rpy="0 ${pi/2} 0" />
-    </link>
+    </link> -->
     <link name="right_wheel_link">
         <visual>
@@ -113,5 +114,6 @@
     <!--<xacro:include filename="$(find my_robot_description)/urdf/pusharm.urdf.xacro">
     <link name="arm1_link" />-->
-        <link name="pusher_arm_link">
+<!--Pushers below, commented out for testing-->
+        <!-- <link name="pusher_arm_link">
         <visual>
             <geometry>
@@ -160,5 +162,5 @@
         </collision>
         <xacro:box_inertia m="2.0" x="${pusher_length}" y="${pusher_width}" z="${pusher_height}" o_xyz="0 0 ${pusher_height/2}" o_rpy="0 0 0" />
-    </link>
+    </link> -->
     <!--Joints here-->
     <!--Joints attach links to each other. DIfferent joint types cause different behaviours. I.E "fixed" disallows movement, would be like welding. COntinuous allows rotation forever. So on.-->
@@ -170,10 +172,11 @@
     </joint>
     <!--My first joint, attaching drill to chassis-->
-    <joint name="base_drill_cone_joint" type="continuous">
+    <!--Drill commented out-->
+    <!-- <joint name="base_drill_cone_joint" type="continuous">
         <parent link="base_link" />
         <child link="drill_cone_link" />
         <origin xyz="${base_length} 0 ${wheel_radius}" rpy="0 0 0" />
         <axis xyz="1 0 0" />
-    </joint>
+    </joint> -->
     <joint name="base_right_wheel_joint" type="continuous">
         <parent link="base_link" />
@@ -198,5 +201,6 @@
         <origin xyz="${base_length/2} ${base_width/2 + pusher_arm_radius} 0" rpy="0 0 0" />
     </joint>-->
-    <joint name="left_pusher_pusher_arm_joint" type="fixed">
+<!--Pusher joints, removed for testing-->
+    <!-- <joint name="left_pusher_pusher_arm_joint" type="fixed">
         <parent link="pusher_arm_link" />
         <child link="left_pusher_link" />
@@ -213,5 +217,5 @@
         <origin xyz="0 0 ${pusher_length/2 + base_height}" rpy="0 -1.571 1.571" />
         <axis xyz="0 0 1" />
-        <limit lower="${-pusher_arm_length}" upper="${pusher_arm_length}" effort="20" velocity="0.5" />
-    </joint>
+        <limit lower="${-pusher_arm_length}" upper="${pusher_arm_length}" effort="20" velocity="0.0" />
+    </joint> -->
 </robot>

File: src/my_robot_description/urdf/my_robot.urdf.xacro (robot description, xacro)
@@ -1,3 +1,3 @@
 version https://git-lfs.github.com/spec/v1
-oid sha256:d818b668b28722f5b6ec0c647ea98d876366c0355e968b1a89370087401d4b68
-size 10397
+oid sha256:b884678daeb92276b85730c0183d2e36823eaac162ee8973383bfadb45f12340
+size 10645
